File: COMM.kicad_pcb (KiCad board)
At the start: 4 copper layers, 90.2 x 95.9 mm, 24 parts, among them IC1 Voltage Converter (ADP7158ARD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, J1 SMA Conn. (RFPC-SMA29-F), SW1 Inhibit Switch (SS5GLD2), U1 AX.25 Module (DMR818SU), U2 XBee Module (XBP9B-DMSTB002)

Commit message: Finished schematic and fully routed PCB.
Signed-off-by: Logan Tolbert <xem6df@virginia.edu>
Parts:
- removed the U1 at (156.3, 85.9)
- added C10: 100 nF, C_100nF:CAPC1608X90, F.Cu at (176.2, 85.0)
- added C11: 100 nF, C_100nF:CAPC1608X90, F.Cu at (181.4, 85.0)
- added C5: 100 nF, C_100nF:CAPC1608X90, F.Cu at (121.7, 111.0)
- added C6: 100 pF, C_100pF:CAPC1005X55N, F.Cu at (109.2, 62.9)
- added C7: 47 μF, C_47uF:CAPC2012X135N, F.Cu at (121.5, 107.3)
- added C8: 100 pF, C_100pF:CAPC1005X55N, F.Cu at (109.1, 64.7)
- added C9: 100 pF, C_100pF:CAPC1005X55N, F.Cu at (121.0, 103.6)
- added D2: Voltage Converter DMR (1N4002), Diode_THT:D_DO-41_SOD81_P10.16mm_Horizontal, F.Cu at (118.8, 91.3)
- added D4: LED, LED_THT:LED_D3.0mm, F.Cu at (109.0, 86.5)
- added L1: 18 nH, LQG15HS18NJ02D_18nH:INDC1005X55N, F.Cu at (184.0, 87.8)
- added L2: 200 nH, CLT32_R20_200nH:IND_CLT32-R20, F.Cu at (173.6, 90.3)
- added L3: 200 nH, CLT32_R20_200nH:IND_CLT32-R20, F.Cu at (167.8, 90.1)
- added R3: 220 Ω, R_10OHM:RESC1005X40, F.Cu at (109.0, 66.8)
- added R4: 10 kΩ, Resistor_SMD:R_0805_2012Metric, F.Cu at (152.0, 105.5)
- added U2: AX.25 Module (DMR818SU), DMR818S:DMR818SU, F.Cu at (168.2, 117.2)
- J1: value SMA Conn. (RFPC-SMA29-F) -> SMA Conn. (RFPC-SMA30-F); footprint RFPC-SMA29-F:GRADCONN_RFPC-SMA29-F -> RFPC-SMA30-F:GRADCONN_RFPC-SMA30-F
- R2: value 10Ω -> 470 Ω
- moved SW1 81.7 mm to (109.8, 94.7), turned to -90 degrees
- moved D1 77.8 mm to (109.3, 72.4), turned to 90 degrees
- moved D3 76.8 mm to (109.0, 77.6)
- moved R1 57.6 mm to (117.4, 110.9), turned to 180 degrees
- moved C12 30.1 mm to (119.6, 75.7)
- moved J1 27.3 mm to (178.8, 77.4), turned to 90 degrees
- moved R2 13.3 mm to (114.8, 80.0), turned to -90 degrees
- moved C13 7.28 mm to (118.3, 77.9), turned to 0 degrees
- moved C1 6.43 mm to (181.3, 70.8)
- moved U1 4.36 mm to (134.0, 124.4)
- moved C2 2.49 mm to (124.7, 143.8)
- moved C3 2.32 mm to (124.7, 141.1)
- moved C4 2.29 mm to (124.9, 138.6)
- moved C14 1.85 mm to (116.5, 88.3)
- moved C15 1.77 mm to (118.8, 88.3)
- renumbered C5 to C12, C6 to C13, C7 to C14, C8 to C15, D2 to D3, U2 to U1
Connections:
- C2 pad 1: Net-(SW1-A) -> +3.3V
- C3 pad 1: Net-(SW1-A) -> +3.3V
- C4 pad 1: Net-(SW1-A) -> +3.3V
- D3 pad 2: Net-(D2-A) -> /Associate/DIO5_XB
- H1 pad 11: /T/R_DMR -> unconnected-(H1-Pad11)
- H1 pad 13: /CS_DMR -> unconnected-(H1-Pad13)
- H1 pad 15: /PTT_DMR -> unconnected-(H1-Pad15)
- H1 pad 17: /HST_TXD_DMR -> unconnected-(H1-Pad17)
- H1 pad 19: /HST_RXD_DMR -> unconnected-(H1-Pad19)
- H1 pad 5: /CTS_XB -> unconnected-(H1-Pad5)
- H1 pad 7: /RTS_XB -> unconnected-(H1-Pad7)
- H1 pad 9: /GPIO_XB -> unconnected-(H1-Pad9)
- H2 pad 1: unconnected-(H2-Pad1) -> /DIN/CONFIG/DIO14_XB
- H2 pad 10: unconnected-(H2-Pad10) -> /AD1/DIO1/SPI_ATTN_XB
- H2 pad 11: unconnected-(H2-Pad11) -> /ON_SLEEP/DIO9_XB
- H2 pad 12: unconnected-(H2-Pad12) -> /DIO10/PWM0_XB
- H2 pad 13: unconnected-(H2-Pad13) -> /RESET_XB
- H2 pad 14: unconnected-(H2-Pad14) -> /DIO11/PWM1_XB
- H2 pad 15: unconnected-(H2-Pad15) -> /AD0/DIO0_XB
- H2 pad 16: unconnected-(H2-Pad16) -> /Associate/DIO5_XB
- H2 pad 17: unconnected-(H2-Pad17) -> /NDTR_XB
- H2 pad 19: unconnected-(H2-Pad19) -> /MIC_IN_DMR
- H2 pad 2: unconnected-(H2-Pad2) -> /DOUT/DIO13_XB
- H2 pad 20: unconnected-(H2-Pad20) -> /LINE_OUT_DMR
- H2 pad 21: unconnected-(H2-Pad21) -> /T/R_DMR
- H2 pad 22: unconnected-(H2-Pad22) -> /PTT_DMR
- H2 pad 23: unconnected-(H2-Pad23) -> /SPKEN_DMR
- H2 pad 24: unconnected-(H2-Pad24) -> /CS_DMR
- H2 pad 25: unconnected-(H2-Pad25) -> /HST_RXD_DMR
- H2 pad 26: unconnected-(H2-Pad26) -> /UART_RX_DMR
- H2 pad 27: unconnected-(H2-Pad27) -> /HST_TXD_DMR
- H2 pad 28: unconnected-(H2-Pad28) -> /UART_TX_DMR
- H2 pad 3: unconnected-(H2-Pad3) -> /RTS/DOI6_XB
- H2 pad 4: unconnected-(H2-Pad4) -> /CTS/DIO7_XB
- H2 pad 5: unconnected-(H2-Pad5) -> /AD3/DIO3/SPI_SSEL_XB
- H2 pad 6: unconnected-(H2-Pad6) -> /AD2/DIO2/SPI_CLK_XB
- H2 pad 7: unconnected-(H2-Pad7) -> /DIO4/SPI_MOSI_XB
- H2 pad 8: unconnected-(H2-Pad8) -> /DIO12/SPI_MISO
- H2 pad 9: unconnected-(H2-Pad9) -> /DTR/SLEEP_RQ/DIO8
- IC1 pad 4: +5V -> /Voltage Converter XB/VIN
- IC1 pad 8: +5V -> /Voltage Converter XB/VIN
- J1 pad 1: Net-(U1-ANT) -> /DMR818S-U 2W RF Module/ANT
- R2 pad 2: Net-(SW1-A) -> /Voltage Converter XB/VIN
- SW1 pad 1: Net-(SW1-A) -> /Voltage Converter XB/VIN
- SW1 pad 2: +3.3V -> +5V
- U1 pad 1: Net-(SW1-A) -> +3.3V
- U1 pad 11: unconnected-(U2-DIO4/SPI_MOSI-Pad11) -> /DIO4/SPI_MOSI_XB
- U1 pad 12: /CTS_XB -> /CTS/DIO7_XB
- U1 pad 13: /SLEEP_XB -> /ON_SLEEP/DIO9_XB
- U1 pad 15: Net-(D2-A) -> /Associate/DIO5_XB
- U1 pad 16: /RTS_XB -> /RTS/DOI6_XB
- U1 pad 17: unconnected-(U2-AD3/DIO3/SPI_NSSEL-Pad17) -> /AD3/DIO3/SPI_SSEL_XB
- U1 pad 18: unconnected-(U2-AD2/DIO2/SPI_CLK-Pad18) -> /AD2/DIO2/SPI_CLK_XB
- U1 pad 19: unconnected-(U2-AD1/DIO1/SPI_NATTN-Pad19) -> /AD1/DIO1/SPI_ATTN_XB
- U1 pad 2: /UART_D_TX -> /DOUT/DIO13_XB
- U1 pad 20: /GPIO_XB -> /AD0/DIO0_XB
- U1 pad 3: /UART_D_RX -> /DIN/CONFIG/DIO14_XB
- U1 pad 4: unconnected-(U2-DIO12/SPI_MISO-Pad4) -> /DIO12/SPI_MISO
- U1 pad 5: /X_RESET -> /RESET_XB
- U1 pad 6: /PWM0_XB -> /DIO10/PWM0_XB
- U1 pad 7: /PWM1_XB -> /DIO11/PWM1_XB
- U1 pad 9: unconnected-(U2-NDTR/SLEEP_RQ/DIO8-Pad9) -> /DTR/SLEEP_RQ/DIO8
Routing:
- net GND: track 0.00 -> 548.1 mm, vias 0 -> 1
- net /Associate/DIO5_XB: track 0.00 -> 121.7 mm
- net +3.3V: track 0.00 -> 115.8 mm
- net /SPKEN_DMR: track 0.00 -> 107.9 mm, vias 0 -> 1
- net /DOUT/DIO13_XB: track 0.00 -> 107.0 mm
- net /AD3/DIO3/SPI_SSEL_XB: track 0.00 -> 104.7 mm
- net /MIC_IN_DMR: track 0.00 -> 104.4 mm
- net /DIN/CONFIG/DIO14_XB: track 0.00 -> 104.4 mm
- net /DIO11/PWM1_XB: track 0.00 -> 102.2 mm
- net /T/R_DMR: track 0.00 -> 99.5 mm, vias 0 -> 1
- net +5V: track 0.00 -> 98.5 mm, vias 0 -> 1
- net /RESET_XB: track 0.00 -> 97.0 mm
- net /DIO10/PWM0_XB: track 0.00 -> 96.8 mm
- net /AD2/DIO2/SPI_CLK_XB: track 0.00 -> 96.7 mm
- net /DIO12/SPI_MISO: track 0.00 -> 93.7 mm
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
Commit message: Added 3D models to all components except DMR module, need to make a 3D model for that one.
Signed-off-by: Logan Tolbert <xem6df@virginia.edu>
Parts:
- R1, R4: footprint Resistor_SMD:R_0805_2012Metric -> R_10kO:RESC1005X40N
- R2: footprint R_10OHM:RESC1005X40 -> R_470O:RESC6332X65N
- R3: footprint R_10OHM:RESC1005X40 -> R_220O:RESC6332X70N
- moved R3 13.6 mm to (121.7, 71.6)
- moved R2 5.14 mm to (115.1, 74.8)
Routing:
- net Net-(D4-A): track 17.9 -> 33.7 mm
- net Net-(D1-A): track 11.7 -> 6.59 mm
- net /Voltage Converter XB/VIN: track 38.4 -> 40.6 mm
- net /T/R_DMR: track 99.5 -> 98.7 mm

Commit message: removed extraneous connections to the XBee and DMR modules on schematic and PCB.
Parts:
- removed C8: 100 pF, C_100pF:CAPC1005X55N
- removed R4: 10 kΩ, R_10kO:RESC1005X40N
Connections:
- net /DTR/SLEEP_RQ/DIO8 renamed /DTR/SLEEP_RQ/DIO8_XB
- H2 pad 10: /AD1/DIO1/SPI_ATTN_XB -> unconnected-(H2-Pad10)
- H2 pad 12: /DIO10/PWM0_XB -> unconnected-(H2-Pad12)
- H2 pad 14: /DIO11/PWM1_XB -> unconnected-(H2-Pad14)
- H2 pad 15: /AD0/DIO0_XB -> unconnected-(H2-Pad15)
- H2 pad 17: /NDTR_XB -> unconnected-(H2-Pad17)
- H2 pad 23: /SPKEN_DMR -> unconnected-(H2-Pad23)
- H2 pad 24: /CS_DMR -> unconnected-(H2-Pad24)
- H2 pad 3: /RTS/DOI6_XB -> unconnected-(H2-Pad3)
- H2 pad 4: /CTS/DIO7_XB -> unconnected-(H2-Pad4)
- H2 pad 5: /AD3/DIO3/SPI_SSEL_XB -> unconnected-(H2-Pad5)
- H2 pad 6: /AD2/DIO2/SPI_CLK_XB -> unconnected-(H2-Pad6)
- H2 pad 7: /DIO4/SPI_MOSI_XB -> unconnected-(H2-Pad7)
- H2 pad 8: /DIO12/SPI_MISO -> unconnected-(H2-Pad8)
- U1 pad 11: /DIO4/SPI_MOSI_XB -> unconnected-(U1-DIO4/SPI_MOSI-Pad11)
- U1 pad 12: /CTS/DIO7_XB -> unconnected-(U1-NCTS/DIO7-Pad12)
- U1 pad 16: /RTS/DOI6_XB -> unconnected-(U1-NRTS/DIO6-Pad16)
- U1 pad 17: /AD3/DIO3/SPI_SSEL_XB -> unconnected-(U1-AD3/DIO3/SPI_NSSEL-Pad17)
- U1 pad 18: /AD2/DIO2/SPI_CLK_XB -> unconnected-(U1-AD2/DIO2/SPI_CLK-Pad18)
- U1 pad 19: /AD1/DIO1/SPI_ATTN_XB -> unconnected-(U1-AD1/DIO1/SPI_NATTN-Pad19)
- U1 pad 20: /AD0/DIO0_XB -> unconnected-(U1-AD0/DIO0-Pad20)
- U1 pad 4: /DIO12/SPI_MISO -> unconnected-(U1-DIO12/SPI_MISO-Pad4)
- U1 pad 6: /DIO10/PWM0_XB -> unconnected-(U1-DIO10/PWM0-Pad6)
- U1 pad 7: /DIO11/PWM1_XB -> unconnected-(U1-DIO11/PWM1-Pad7)
- U2 pad 13: Net-(U2-CS) -> unconnected-(U2-CS-Pad13)
- U2 pad 18: /SPKEN_DMR -> unconnected-(U2-SPKEN-Pad18)
Routing:
- net /SPKEN_DMR: track 108.3 -> 0.00 mm, vias 1 -> 0
- net /AD3/DIO3/SPI_SSEL_XB: track 104.7 -> 0.00 mm
- net /DIO11/PWM1_XB: track 102.2 -> 0.00 mm
- net /DIO10/PWM0_XB: track 96.8 -> 0.00 mm
- net /AD2/DIO2/SPI_CLK_XB: track 96.7 -> 0.00 mm
- net /DIO12/SPI_MISO: track 93.7 -> 0.00 mm
- net /RTS/DOI6_XB: track 91.3 -> 0.00 mm
- net /AD1/DIO1/SPI_ATTN_XB: track 81.6 -> 0.00 mm
- net /AD0/DIO0_XB: track 78.7 -> 0.00 mm
- net /CTS/DIO7_XB: track 65.5 -> 0.00 mm
- net /DIO4/SPI_MOSI_XB: track 60.3 -> 0.00 mm
- net /CS_DMR: track 45.3 -> 0.00 mm
- net /T/R_DMR: track 98.7 -> 88.1 mm
- net Net-(U2-CS): track 3.78 -> 0.00 mm
- net GND: track 548.4 -> 546.6 mm
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
Commit message: Corrected DMR footprint and adjusted some routing.
Signed-off-by: Logan Tolbert <xem6df@virginia.edu>
Parts:
- moved U2 0.19 mm to (168.2, 117.1)
Routing:
- net /T/R_DMR: track 88.1 -> 90.6 mm
- net Net-(U2-UART_TX): track 46.3 -> 48.7 mm
- net Net-(U2-UART_RX): track 37.8 -> 39.9 mm
- net /MIC_IN_DMR: track 103.7 -> 101.8 mm
- net +3.3V: track 115.2 -> 113.6 mm
- net /HST_TXD_DMR: track 58.9 -> 58.2 mm
- net /LINE_OUT_DMR: track 64.5 -> 63.9 mm
- net GND: track 546.6 -> 546.1 mm

Commit message: Added pull-up to CS pin on DMR module.
Signed-off-by: Logan Tolbert <xem6df@virginia.edu>
Parts:
- added R4: 10 kΩ, R_10kO:RESC1005X40N, F.Cu at (152.5, 105.0)
- renumbered C11 to C10, C12 to C11, C13 to C12, C14 to C13, C15 to C14, C9 to C8, C10 to C9
Connections:
- U2 pad 13: unconnected-(U2-CS-Pad13) -> Net-(U2-CS)
Routing:
- net /DMR818S-U 2W RF Module/VCC: track 63.8 -> 76.8 mm, vias 2 -> 1
- net Net-(U2-CS): track 0.00 -> 3.99 mm
- net +5V: track 98.5 -> 102.0 mm
