File: TPS61085.kicad_sch (KiCad schematic)
At the start: 11 parts, among them U3 TPS61085PWR

Commit message: Finalized board design, updated DMR module to DMR818S-5W exact dimensions, rerouted PCB according to McPherson's comments. Added TLV61047 5V to 8V booster module.
Signed-off-by: Logan Tolbert <xem6df@virginia.edu>
Parts:
- C12: footprint (none) -> C_100nF:CAPC1608X90
- C13: footprint (none) -> Capacitor_SMD:C_0603_1608Metric
- C14: footprint (none) -> C_1uF:CAPC1005X55N
- C15, C16: footprint (none) -> C_10uF:CAPC1005X70N
- L2: footprint (none) -> Inductor_SMD:L_0805_2012Metric
- R5, R6, R7: footprint (none) -> Resistor_SMD:R_1210_3225Metric
Changed lines of the file:
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@@
 			)
 		)
-		(property "Footprint" ""
+		(property "Footprint" "C_100nF:CAPC1608X90"
 			(at 104.4448 82.55 0)
 			(effects
@@
 			)
 		)
-		(property "Footprint" ""
+		(property "Footprint" "C_1uF:CAPC1005X55N"
 			(at 176.2252 66.04 0)
 			(effects
@@
 			)
 		)
-		(property "Footprint" ""
+		(property "Footprint" "C_10uF:CAPC1005X70N"
 			(at 192.7352 97.79 0)
 			(effects
@@
 			)
 		)
-		(property "Footprint" ""
+		(property "Footprint" "Resistor_SMD:R_1210_3225Metric"
 			(at 162.306 99.314 90)
 			(effects
@@
 			)
 		)
-		(property "Footprint" ""
+		(property "Footprint" "C_10uF:CAPC1005X70N"
 			(at 174.2948 123.19 0)
 			(effects
@@
 			)
 		)
-		(property "Footprint" ""
+		(property "Footprint" "Resistor_SMD:R_1210_3225Metric"
 			(at 147.574 120.904 90)
 			(effects
@@
 			)
 		)
-		(property "Footprint" ""
+		(property "Footprint" "Capacitor_SMD:C_0603_1608Metric"
 			(at 162.2552 110.49 0)
 			(effects
@@
 			)
 		)
-		(property "Footprint" ""
+		(property "Footprint" "Resistor_SMD:R_1210_3225Metric"
 			(at 119.126 127.254 90)
 			(effects
@@
 			)
 		)
-		(property "Footprint" ""
+		(property "Footprint" "Inductor_SMD:L_0805_2012Metric"
 			(at 184.15 88.9 0)
 			(effects
