File: voltageStepDMR.kicad_sch (KiCad schematic)
At the start: 8 parts, among them IC1 TLV61047DDCR

Commit message: Final COMM board design as of Feb 12 2026, ready to order.
Signed-off-by: Logan Tolbert <xem6df@virginia.edu>
Parts:
- D5: footprint Diode_SMD:Nexperia_CFP3_SOD-123W -> PMEG3020BER_115:DIODE_SOD123W_1P9X2P8_NEX
- renumbered C13 to C10, C14 to C11, C12 to C9, L2 to L1
Changed lines of the file:
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@@
 		(dnp no)
 		(fields_autoplaced yes)
-		(property "Reference" "#PWR036"
+		(property "Reference" "#PWR034"
 			(at 198.12 110.49 0)
 			(effects
@@
 			(project "COMM"
 				(path "/b0bd204d-ca77-4624-acd2-31813bf00a6c/0fe138ce-d52b-4e48-afd9-f8e26f885e70"
-					(reference "#PWR036")
+					(reference "#PWR034")
 					(unit 1)
 				)
@@
 		(dnp no)
 		(fields_autoplaced yes)
-		(property "Reference" "C13"
+		(property "Reference" "C10"
 			(at 176.53 80.0099 0)
 			(effects
@@
 			(project "COMM"
 				(path "/b0bd204d-ca77-4624-acd2-31813bf00a6c/0fe138ce-d52b-4e48-afd9-f8e26f885e70"
-					(reference "C13")
+					(reference "C10")
 					(unit 1)
 				)
@@
 		(dnp no)
 		(fields_autoplaced yes)
-		(property "Reference" "#PWR032"
+		(property "Reference" "#PWR030"
 			(at 120.65 91.44 0)
 			(effects
@@
 			(project "COMM"
 				(path "/b0bd204d-ca77-4624-acd2-31813bf00a6c/0fe138ce-d52b-4e48-afd9-f8e26f885e70"
-					(reference "#PWR032")
+					(reference "#PWR030")
 					(unit 1)
 				)
@@
 		(dnp no)
 		(fields_autoplaced yes)
-		(property "Reference" "L2"
+		(property "Reference" "L1"
 			(at 139.7 69.85 90)
 			(effects
@@
 			(project ""
 				(path "/b0bd204d-ca77-4624-acd2-31813bf00a6c/0fe138ce-d52b-4e48-afd9-f8e26f885e70"
-					(reference "L2")
+					(reference "L1")
 					(unit 1)
 				)
@@
 		(dnp no)
 		(fields_autoplaced yes)
-		(property "Reference" "#PWR033"
+		(property "Reference" "#PWR031"
 			(at 158.75 92.71 0)
 			(effects
@@
 			(project ""
 				(path "/b0bd204d-ca77-4624-acd2-31813bf00a6c/0fe138ce-d52b-4e48-afd9-f8e26f885e70"
-					(reference "#PWR033")
+					(reference "#PWR031")
 					(unit 1)
 				)
@@
 		(on_board yes)
 		(dnp no)
-		(property "Reference" "C12"
+		(property "Reference" "C9"
 			(at 116.84 80.0099 0)
 			(effects
@@
 			(project ""
 				(path "/b0bd204d-ca77-4624-acd2-31813bf00a6c/0fe138ce-d52b-4e48-afd9-f8e26f885e70"
-					(reference "C12")
+					(reference "C9")
 					(unit 1)
 				)
@@
 		(dnp no)
 		(fields_autoplaced yes)
-		(property "Reference" "#PWR034"
+		(property "Reference" "#PWR032"
 			(at 172.72 91.44 0)
 			(effects
@@
 			(project "COMM"
 				(path "/b0bd204d-ca77-4624-acd2-31813bf00a6c/0fe138ce-d52b-4e48-afd9-f8e26f885e70"
-					(reference "#PWR034")
+					(reference "#PWR032")
 					(unit 1)
 				)
@@
 		(dnp no)
 		(fields_autoplaced yes)
-		(property "Reference" "C14"
+		(property "Reference" "C11"
 			(at 189.23 80.0099 0)
 			(effects
@@
 			(project "COMM"
 				(path "/b0bd204d-ca77-4624-acd2-31813bf00a6c/0fe138ce-d52b-4e48-afd9-f8e26f885e70"
-					(reference "C14")
+					(reference "C11")
 					(unit 1)
 				)
@@
 			)
 		)
-		(property "Footprint" "Diode_SMD:Nexperia_CFP3_SOD-123W"
+		(property "Footprint" "PMEG3020BER_115:DIODE_SOD123W_1P9X2P8_NEX"
 			(at 163.83 71.755 0)
 			(effects
@@
 		(dnp no)
 		(fields_autoplaced yes)
-		(property "Reference" "#PWR035"
+		(property "Reference" "#PWR033"
 			(at 185.42 91.44 0)
 			(effects
@@
 			(project "COMM"
 				(path "/b0bd204d-ca77-4624-acd2-31813bf00a6c/0fe138ce-d52b-4e48-afd9-f8e26f885e70"
-					(reference "#PWR035")
-					(unit 1)
-				)
+					(reference "#PWR033")
+					(unit 1)
+				)
